Commit message: add slam_toolbox and nav2

File: src/wheebot_description/urdf/wheebot_ros2_control.xacro (robot description, xacro)
@@ -20,5 +20,5 @@
             </hardware>
         </xacro:unless>
-        <joint name="wheel_right_joint">
+        <joint name="wheel_left_joint">
             <command_interface name="velocity">
                 <param name="min">-1</param>
@@ -28,5 +28,5 @@
             <state_interface name="velocity"/>
         </joint>
-        <joint name="wheel_left_joint">
+        <joint name="wheel_right_joint">
             <command_interface name="velocity">
                 <param name="min">-1</param>
