Commit message: add sensors

File: src/wheebot_description/urdf/wheebot.urdf.xacro (robot description, xacro)
@@ -2,4 +2,5 @@
 <robot xmlns:xacro="http://www.ros.org/wiki/xacro" name="wheebot">
     <xacro:arg name="is_ignition" default="true" />
+    <xacro:arg name="is_sim" default="true"/>
     <!-- Include Gazebo Parameters -->
     <xacro:include filename="$(find wheebot_description)/urdf/wheebot_gazebo.xacro" />
@@ -21,4 +22,5 @@
                 <mesh filename="package://wheebot_description/meshes/wheebot_base_link.stl" scale="0.001 0.001 0.001"/>
             </geometry>
+            <material name="silver"/>
         </visual>
         <collision>
@@ -49,4 +51,5 @@
                 <mesh filename="package://wheebot_description/meshes/wheebot_wheel_link.stl" scale="0.001 0.001 0.001"/>
             </geometry>
+            <material name="black"/>
         </visual>
         <collision>
@@ -80,4 +83,5 @@
                 <mesh filename="package://wheebot_description/meshes/wheebot_wheel_link.stl" scale="0.001 0.001 0.001"/>
             </geometry>
+            <material name="black"/>
         </visual>
         <collision>
@@ -110,4 +114,5 @@
                 <mesh filename="package://wheebot_description/meshes/wheebot_caster_fork_link.stl" scale="0.001 0.001 0.001"/>
             </geometry>
+            <material name="silver"/>
         </visual>
         <collision>
@@ -139,4 +144,5 @@
                 <mesh filename="package://wheebot_description/meshes/wheebot_caster_wheel_link.stl" scale="0.001 0.001 0.001"/>
             </geometry>
+            <material name="black"/>
         </visual>
         <collision>
@@ -169,4 +175,5 @@
                 <mesh filename="package://wheebot_description/meshes/wheebot_caster_fork_link.stl" scale="0.001 0.001 0.001"/>
             </geometry>
+            <material name="silver"/>
         </visual>
         <collision>
@@ -198,4 +205,5 @@
                 <mesh filename="package://wheebot_description/meshes/wheebot_caster_wheel_link.stl" scale="0.001 0.001 0.001"/>
             </geometry>
+            <material name="black"/>
         </visual>
         <collision>
@@ -227,4 +235,8 @@
                 <mesh filename="package://wheebot_description/meshes/imu_link.STL"/>
             </geometry>
+            <material name="">
+                <color rgba="0.792156862745098 0.819607843137255 0.933333333333333 1" />
+            </material>
+            <material name="blue"/>
         </visual>
         <collision>
@@ -241,3 +253,48 @@
         <axis xyz="0 0 0"/>
     </joint>
+    <link name="laser_link">
+        <inertial>
+            <origin xyz="-0.011945780406062 -0.000381929217680526 -0.0170649378129477" rpy="0 0 0" />
+            <mass value="0.073084435549317" />
+            <inertia ixx="1.96074931730795E-05" ixy="-3.62091076640009E-07" ixz="4.28230084046735E-07"
+                     iyy="2.40983835136327E-05" iyz="1.50180909250652E-08"
+                     izz="4.14184164228595E-05" />
+        </inertial>
+        <visual>
+            <origin xyz="0 0 0" rpy="0 0 0"/>
+            <geometry>
+                <mesh filename="package://wheebot_description/meshes/laser_link.STL"/>
+            </geometry>
+            <material name="dark_grey"/>
+        </visual>
+        <collision>
+            <origin xyz="0 0 0" rpy="0 0 0"/>
+            <geometry>
+                <mesh filename="package://wheebot_description/meshes/laser_link.STL"/>
+            </geometry>
+        </collision>
+    </link>
+    <joint name="laser_joint" type="fixed">
+        <origin rpy="0 0 3.14" xyz="0 0 0.7"/>
+        <parent link="base_link"/>
+        <child link="laser_link"/>
+        <axis xyz="0 0 0" />
+    </joint>
+    <material name="blue">
+        <color rgba="0 0 1 1"/>
+    </material>
+    <material name="black">
+        <color rgba="0 0 0 1"/>
+    </material>
+    <material name="silver">
+        <color rgba="0.79 0.82 0.93 1"/>
+    </material>
+    <material name="dark_grey">
+        <color rgba="0.3 0.3 0.3 1"/>
+    </material>
+    <xacro:arg name="use_nominal_extrinsics" default="false" />
+    <xacro:include filename="$(find realsense2_description)/urdf/_d435i.urdf.xacro"/>
+    <xacro:sensor_d435i parent="base_link" use_nominal_extrinsics="$(arg use_nominal_extrinsics)">
+        <origin xyz="0 0 0.63" rpy="0 0 0"/>
+    </xacro:sensor_d435i>
 </robot>

File: src/wheebot_description/urdf/wheebot_gazebo.xacro (robot description, xacro)
@@ -42,4 +42,7 @@
             <plugin filename="ignition-gazebo-imu-system" name="ignition::gazebo::systems::Imu">
             </plugin>
+            <plugin filename="ignition-gazebo-sensors-system" name="ignition::gazebo::systems::Sensors">
+                <render_engine>ogre2</render_engine>
+            </plugin>
         </xacro:if>
         <xacro:unless value="$(arg is_ignition)">
@@ -48,4 +51,7 @@
             </plugin>
             <plugin filename="gz-sim-imu-system" name="gz::sim::systems::Imu">
+            </plugin>
+            <plugin filename="gz-sim-sensors-system" name="gz::sim::systems::Sensors">
+                <render_engine>ogre2</render_engine>
             </plugin>
         </xacro:unless>
@@ -101,3 +107,70 @@
         </sensor>
     </gazebo>
+    <gazebo reference="laser_link">
+        <sensor name="lidar" type="gpu_lidar">
+            <always_on>true</always_on>
+            <visualize>true</visualize>
+            <topic>scan</topic>
+            <update_rate>5</update_rate>
+            <gz_frame_id>laser_link</gz_frame_id>
+            <lidar>
+                <scan>
+                    <horizontal>
+                    <samples>360</samples>
+                    <resolution>1.00000</resolution>
+                    <min_angle>0.000000</min_angle>
+                    <max_angle>6.280000</max_angle>
+                    </horizontal>
+                </scan>
+                <range>
+                    <min>0.120000</min>
+                    <max>12.0</max>
+                    <resolution>0.02</resolution>
+                </range>
+                <noise>
+                    <type>gaussian</type>
+                    <mean>0.0</mean>
+                    <stddev>0.01</stddev>
+                </noise>
+            </lidar>
+        </sensor>
+    </gazebo>
+    <gazebo reference="camera_link">
+        <sensor name="rgbd_camera" type="rgbd_camera">
+            <camera>
+                <horizontal_fov>1.05</horizontal_fov>
+                <image>
+                    <width>640</width>
+                    <height>480</height>
+                </image>
+                <clip>
+                    <near>0.1</near>
+                    <far>10.0</far>
+                </clip>
+            </camera>
+            <always_on>true</always_on>
+            <gz_frame_id>camera_link</gz_frame_id>
+            <topic>camera</topic>
+            <update_rate>30</update_rate>
+            <visualize>true</visualize>
+        </sensor>
+        <sensor name="imu_camera" type="imu">
+            <always_on>true</always_on>
+            <update_rate>200</update_rate>
+            <topic>camera/imu</topic>
+            <gz_frame_id>camera_link</gz_frame_id>
+            <imu>
+                <angular_velocity>
+                    <x><noise type="gaussian"><mean>0.0</mean><stddev>2e-4</stddev></noise></x>
+                    <y><noise type="gaussian"><mean>0.0</mean><stddev>2e-4</stddev></noise></y>
+                    <z><noise type="gaussian"><mean>0.0</mean><stddev>2e-4</stddev></noise></z>
+                </angular_velocity>
+                <linear_acceleration>
+                    <x><noise type="gaussian"><mean>0.0</mean><stddev>1.7e-2</stddev></noise></x>
+                    <y><noise type="gaussian"><mean>0.0</mean><stddev>1.7e-2</stddev></noise></y>
+                    <z><noise type="gaussian"><mean>0.0</mean><stddev>1.7e-2</stddev></noise></z>
+                </linear_acceleration>
+            </imu>
+        </sensor>
+    </gazebo>
 </robot>

File: src/wheebot_description/urdf/wheebot_ros2_control.xacro (robot description, xacro)
@@ -2,12 +2,20 @@
 <robot xmlns:xacro="http://www.ros.org/wiki/xacro" name="wheebot">
     <ros2_control name="RobotSystem" type="system">
-        <xacro:if value="$(arg is_ignition)">
+        <xacro:if value="$(arg is_sim)">
+            <xacro:if value="$(arg is_ignition)">
+                <hardware>
+                    <plugin>ign_ros2_control/IgnitionSystem</plugin>
+                </hardware>
+            </xacro:if>
+            <xacro:unless value="$(arg is_ignition)">
+                <hardware>
+                    <plugin>gz_ros2_control/GazeboSimSystem</plugin>
+                </hardware>
+            </xacro:unless>
+        </xacro:if>
+        <xacro:unless value="$(arg is_sim)">
             <hardware>
-                <plugin>ign_ros2_control/IgnitionSystem</plugin>
-            </hardware>
-        </xacro:if>
-        <xacro:unless value="$(arg is_ignition)">
-            <hardware>
-                <plugin>gz_ros2_control/GazeboSimSystem</plugin>
+                <plugin>wheebot_firmware/WheebotInterface</plugin>
+                <param name="port">/dev/ttyUSB0</param>
             </hardware>
         </xacro:unless>

Commit message: optimize functionalities

File: src/wheebot_description/urdf/wheebot.urdf.xacro (robot description, xacro)
@@ -276,5 +276,8 @@
     </link>
     <joint name="laser_joint" type="fixed">
-        <origin rpy="0 0 3.14" xyz="0 0 0.7"/>
+        <!-- atas -->
+        <!-- <origin rpy="0 0 0" xyz="0 0 0.7"/> -->
+        <!-- armrest -->
+        <origin rpy="0 0 0" xyz="0.3036 0.2157 0.4"/>
         <parent link="base_link"/>
         <child link="laser_link"/>
@@ -296,5 +299,14 @@
     <xacro:include filename="$(find realsense2_description)/urdf/_d435i.urdf.xacro"/>
     <xacro:sensor_d435i parent="base_link" use_nominal_extrinsics="$(arg use_nominal_extrinsics)">
-        <origin xyz="0 0 0.63" rpy="0 0 0"/>
+        <!-- atas -->
+        <!-- <origin xyz="0.058 0 0.638" rpy="0 0 0"/> -->
+        <!-- armrest -->
+        <origin xyz="0.3616 0.2157 0.338" rpy="0 0 0"/>
     </xacro:sensor_d435i>
+    <link name="camera_optical_frame"/>
+    <joint name="camera_optical_joint" type="fixed">
+    <parent link="camera_link"/>
+    <child link="camera_optical_frame"/>
+    <origin xyz="0 0 0" rpy="-1.5708 0 -1.5708"/>
+    </joint>
 </robot>

File: src/wheebot_description/urdf/wheebot_gazebo.xacro (robot description, xacro)
@@ -65,42 +65,12 @@
             <imu>
                 <angular_velocity>
-                    <x>
-                        <noise type="gaussian">
-                            <mean>0.0</mean>
-                            <stddev>2e-4</stddev>
-                        </noise>
-                    </x>
-                    <y>
-                        <noise type="gaussian">
-                            <mean>0.0</mean>
-                            <stddev>2e-4</stddev>
-                        </noise>
-                    </y>
-                    <z>
-                        <noise type="gaussian">
-                            <mean>0.0</mean>
-                            <stddev>2e-4</stddev>
-                        </noise>
-                    </z>
+                    <x><noise type="gaussian"><mean>0.0</mean><stddev>2e-4</stddev></noise></x>
+                    <y><noise type="gaussian"><mean>0.0</mean><stddev>2e-4</stddev></noise></y>
+                    <z><noise type="gaussian"><mean>0.0</mean><stddev>2e-4</stddev></noise></z>
                 </angular_velocity>
                 <linear_acceleration>
-                    <x>
-                        <noise type="gaussian">
-                            <mean>0.0</mean>
-                            <stddev>1.7e-2</stddev>
-                        </noise>
-                    </x>
-                    <y>
-                        <noise type="gaussian">
-                            <mean>0.0</mean>
-                            <stddev>1.7e-2</stddev>
-                        </noise>
-                    </y>
-                    <z>
-                        <noise type="gaussian">
-                            <mean>0.0</mean>
-                            <stddev>1.7e-2</stddev>
-                        </noise>
-                    </z>
+                    <x><noise type="gaussian"><mean>0.0</mean><stddev>1.7e-2</stddev></noise></x>
+                    <y><noise type="gaussian"><mean>0.0</mean><stddev>1.7e-2</stddev></noise></y>
+                    <z><noise type="gaussian"><mean>0.0</mean><stddev>1.7e-2</stddev></noise></z>
                 </linear_acceleration>
             </imu>
@@ -111,25 +81,26 @@
             <always_on>true</always_on>
             <visualize>true</visualize>
+            <!-- <pose relative_to='laser_link'>0 0 0 0 0 0</pose> -->
+            <gz_frame_id>laser_link</gz_frame_id>
             <topic>scan</topic>
-            <update_rate>5</update_rate>
-            <gz_frame_id>laser_link</gz_frame_id>
+            <update_rate>3</update_rate>
             <lidar>
                 <scan>
                     <horizontal>
-                    <samples>360</samples>
-                    <resolution>1.00000</resolution>
-                    <min_angle>0.000000</min_angle>
-                    <max_angle>6.280000</max_angle>
+                        <samples>720</samples>
+                        <resolution>1.00000</resolution>
+                        <min_angle>-3.14</min_angle>
+                        <max_angle>3.14</max_angle>
                     </horizontal>
                 </scan>
                 <range>
-                    <min>0.120000</min>
+                    <min>0.1</min>
                     <max>12.0</max>
-                    <resolution>0.02</resolution>
+                    <resolution>0.005</resolution>
                 </range>
                 <noise>
                     <type>gaussian</type>
                     <mean>0.0</mean>
-                    <stddev>0.01</stddev>
+                    <stddev>0.001</stddev>
                 </noise>
             </lidar>
@@ -150,5 +121,5 @@
             </camera>
             <always_on>true</always_on>
-            <gz_frame_id>camera_link</gz_frame_id>
+            <gz_frame_id>camera_optical_frame</gz_frame_id>
             <topic>camera</topic>
             <update_rate>30</update_rate>
@@ -157,5 +128,5 @@
         <sensor name="imu_camera" type="imu">
             <always_on>true</always_on>
-            <update_rate>200</update_rate>
+            <update_rate>100</update_rate>
             <topic>camera/imu</topic>
             <gz_frame_id>camera_link</gz_frame_id>
